File: MiniDox.sch (KiCad schematic (older format))
At the start: 41 parts, among them K1 KEYSW, K10 KEYSW, K11 KEYSW, K12 KEYSW, K13 KEYSW, K14 KEYSW, K15 KEYSW, K16 KEYSW, K17 KEYSW, K18 KEYSW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

Commit message: remove pro micro from schematic
Parts:
- removed U1: ProMicro, canadian_footprints:Pro_Micro, symbol ProMicro
- added C? (x2): 10uF, symbol device:CP1_Small
- added C? (x2): 1uF, symbol device:C_Small
- added C? (x2): 0.1uF, symbol device:C_Small
- added C? (x2): 22pF, symbol device:C_Small
- added D?: D_Small, symbol device:D_Small
- added D?: Red, symbol device:LED_Small
- added F?: 500mA, symbol device:Polyfuse_Small
- added J?: USB_B_Micro, symbol Connector:USB_B_Micro
- added R?: 10k, symbol device:R_Small
- added R? (x2): 22, symbol device:R_Small
- added R?: 1k, symbol device:R_Small
- added R?: 180, symbol device:R_Small
- added U?: ATMEGA32U4-AU, TQFP44, symbol atmel:ATMEGA32U4-AU
- added U?: MIC5219-5.0, TO_SOT_Packages_SMD:SOT-23-5, symbol regul:MIC5219-5.0
- added Y?: 16MHz, symbol device:Crystal_Small
- D1, D10, D11, D12, D13, D14, D15, D16, D17, D18, D2, D3, D4, D5, D6, D7, D8, D9: symbol D -> device:D
- K1, K10, K11, K12, K13, K14, K15, K16, K17, K18, K2, K3, K4, K5, K6, K7, K8, K9: symbol KEYSW -> MiniDox-rescue:KEYSW-RESCUE-MiniDox
- K19: symbol TRRS_Through-Hole -> MiniDox-rescue:TRRS_Through-Hole-RESCUE-MiniDox
- RESET1: symbol SW_PUSH -> MiniDox-rescue:SW_PUSH-RESCUE-MiniDox
- SJ1, SJ2: symbol SOLDER_JUMPER_3 -> MiniDox-rescue:SOLDER_JUMPER_3-RESCUE-MiniDox
Connections:
- net labels added: D+, D-, RGB_DI, VBUS, VCCQ, reset, speaker
- wire segments 53 -> 176
- no-connect marks 0 -> 15
